File: pcb/VeryCoolUsbHub.kicad_sch (KiCad schematic)
At the start: 33 parts, among them X1 X322525MSB4SI, X2 X322525MSB4SI

Commit message: update
Parts:
- removed R1, R2: 0402WGF5101TCE, EasyEDA:R0402, symbol EasyEDA:0402WGF5101TCE
- added C20, C21, C22: CC0603KRX7R9BB104, EasyEDA:C0603, symbol EasyEDA:CC0603KRX7R9BB104
- added R1: RT1206BRE07900KL, EasyEDA:R1206, symbol EasyEDA:RT1206BRE07900KL
- added R2: RC0402FR-0710KL, EasyEDA:R0402, symbol EasyEDA:RC0402FR-0710KL
- added R7, R8: RC0603FR-07200KL, EasyEDA:R0603, symbol EasyEDA:RC0603FR-07200KL
- added U2: HD3SS3220RNHR, EasyEDA:WQFN-30_L4.5-W2.5-P0.4-BL-EP, symbol EasyEDA:HD3SS3220RNHR
Connections:
- net DN0: no longer USBC_IN1.A7 (DN1), USBC_IN1.B7 (DN2)
- net DN3: no longer ETHERNET_CONTROLLER1.17 (U2DM)
- net DN4: now also ETHERNET_CONTROLLER1.17 (U2DM)
- net DP0: no longer USBC_IN1.A6 (DP1), USBC_IN1.B6 (DP2)
- net GND: now also C22.1, U2.12 (ENn_MUX), U2.13 (GND), U2.22 (ADDR), U2.28 (GND), U2.29 (ENn_CC)
- net RXn0: now also U2.10 (RXn); no longer USBC_IN1.A10 (SSRXn2), USBC_IN1.B10 (SSRXn1)
- net RXp0: now also U2.9 (RXp); no longer USBC_IN1.A11 (SSRXp2), USBC_IN1.B11 (SSRXp1)
- net Txn0: now also U2.7 (TXn); no longer USBC_IN1.A3 (SSTXn1), USBC_IN1.B3 (SSTXn2)
- net Txp0: now also U2.6 (TXp); no longer USBC_IN1.A2 (SSTXP1), USBC_IN1.B2 (SSTXp2)
- net V3.3: now also R7.1, U2.8 (VCC33)
- net VBUS: now also C22.2, R1.1, R2.2, R8.1, U2.30 (VDD5)
- net USBC_IN_CC1: now reaches USBC_IN1.A5 (CC1)
- net USBC_IN_CC1: now also U2.2 (CC1)
- net USBC_IN_CC2: now reaches USBC_IN1.B5 (CC2)
- net USBC_IN_CC2: now also U2.1 (CC2)
- new net: C20.2, U2.21 (TX2p)
- new net: C21.2, U2.20 (TX2n)
- new net: R7.2, U2.11 (DIR)
- new net: R2.1, U2.3 (CURRENT_MODE)
- new net: R1.2, U2.5 (VBUS_DET)
- new net: R8.2, U2.4 (PORT)
- new net USBC_IN_DN1: USBC_IN1.A7 (DN1)
- new net USBC_IN_DN2: USBC_IN1.B7 (DN2)
- new net USBC_IN_DP1: USBC_IN1.A6 (DP1)
- new net USBC_IN_DP2: USBC_IN1.B6 (DP2)
- new net USBC_IN_RXN1: U2.14 (RX1n), USBC_IN1.B10 (SSRXn1)
- new net USBC_IN_RXN2: U2.18 (RX2n), USBC_IN1.A10 (SSRXn2)
- new net USBC_IN_RXP1: U2.15 (RX1p), USBC_IN1.B11 (SSRXp1)
- new net USBC_IN_RXP2: U2.19 (RX2p), USBC_IN1.A11 (SSRXp2)
- new net USBC_IN_TXN1: U2.16 (TX1n), USBC_IN1.A3 (SSTXn1)
- new net USBC_IN_TXN2: C21.1, USBC_IN1.B3 (SSTXn2)
- new net USBC_IN_TXP1: U2.17 (TX1p), USBC_IN1.A2 (SSTXP1)
- new net USBC_IN_TXP2: C20.1, USBC_IN1.B2 (SSTXp2)
- no-connect marks 43 -> 51
Other:
- moved on the sheet: C1, C2, C3, C4, C9, USBC_IN1

Commit message: do a lot of things
Parts:
- removed C9: CL10A106KP8NNNC, EasyEDA:C0603, symbol EasyEDA:CL10A106KP8NNNC
- removed R2: RC0402FR-0710KL, EasyEDA:R0402, symbol EasyEDA:RC0402FR-0710KL
- removed R4, R5: 0402WGF5602TCE, EasyEDA:R0402, symbol EasyEDA:0402WGF5602TCE
- removed R8: RC0603FR-07200KL, EasyEDA:R0603, symbol EasyEDA:RC0603FR-07200KL
- removed USBC_IN1, USBC_OUT1: TYPE-C-31-M-04, EasyEDA:USB-C-SMD_TYPE-C-USB-20, symbol EasyEDA:TYPE-C-31-M-04
- added C19, C23, C24, C29, C30, C31, C32, C9: CC0603KRX7R9BB104, EasyEDA:C0603, symbol EasyEDA:CC0603KRX7R9BB104
- added C28: CL10A106KP8NNNC, EasyEDA:C0603, symbol EasyEDA:CL10A106KP8NNNC
- added R10: RC0402FR-0710KL, EasyEDA:R0402, symbol EasyEDA:RC0402FR-0710KL
- added R11, R12: RC0603FR-07200KL, EasyEDA:R0603, symbol EasyEDA:RC0603FR-07200KL
- added R8: MCR01MZPF4701, EasyEDA:R0402, symbol EasyEDA:MCR01MZPF4701
- added R9: RT1206BRE07900KL, EasyEDA:R1206, symbol EasyEDA:RT1206BRE07900KL
- added U1: HD3SS3220RNHR, EasyEDA:WQFN-30_L4.5-W2.5-P0.4-BL-EP, symbol EasyEDA:HD3SS3220RNHR
- added USBC_IN_1, USBC_OUT_1: TYPE-C-G05-1TDW, EasyEDA:USB-C-SMD_TYPE-C-G05-1TDW, symbol EasyEDA:TYPE-C-G05-1TDW
Connections:
- net DN0: now also USBC_IN_1.A7 (DN1), USBC_IN_1.B7 (DN2)
- net DN3: now also USBC_OUT_1.A7 (DN1), USBC_OUT_1.B7 (DN2)
- net DP0: now also USBC_IN_1.A6 (DP1), USBC_IN_1.B6 (DP2)
- net DP3: now also USBC_OUT_1.A6 (DP1), USBC_OUT_1.B6 (DP2)
- net GND: now also C2.2, C4.2, C19.1, C28.2, C29.1, C30.2, C31.1, C32.2, R8.1, U1.12 (ENn_MUX), U1.13 (GND), U1.22 (ADDR), U1.28 (GND), U1.29 (ENn_CC), USBC_IN_1.A1 (GND), USBC_IN_1.A12 (GND), USBC_IN_1.B1 (GND), USBC_IN_1.B12 (GND), USBC_OUT_1.A1 (GND), USBC_OUT_1.A12 (GND), USBC_OUT_1.B1 (GND), USBC_OUT_1.B12 (GND); no longer C2.1, C4.1, C8.2
- net RXn3: now also U1.10 (RXn)
- net RXp3: now also U1.9 (RXp)
- net Txn3: now also U1.7 (TXn)
- net Txp3: now also U1.6 (TXp)
- net USBC_IN_CC1: now also USBC_IN_1.A5 (CC1)
- net USBC_IN_CC2: now also USBC_IN_1.B5 (CC2)
- net USBC_IN_RXN1: now also USBC_IN_1.B10 (SSRXn1)
- net USBC_IN_RXN2: now also USBC_IN_1.A10 (SSRXn2)
- net USBC_IN_RXP1: now also USBC_IN_1.B11 (SSRXp1)
- net USBC_IN_RXP2: now also USBC_IN_1.A11 (SSRXp2)
- net USBC_IN_TXN1: now also C8.1, USBC_IN_1.A3 (SSTXn1); no longer U2.16 (TX1n)
- net USBC_IN_TXN2: now also USBC_IN_1.B3 (SSTXn2)
- net USBC_IN_TXP1: now also C9.2, USBC_IN_1.A2 (SSTXp1); no longer U2.17 (TX1p)
- net USBC_IN_TXP2: now also USBC_IN_1.B2 (SSTXp2)
- net V3.3: now also R12.1, U1.8 (VCC33)
- net VBUS: now also C2.1, C4.1, C19.2, C28.1, C29.2, C30.1, C31.2, C32.1, R10.2, R11.1, R9.1, U1.30 (VDD5), USBC_IN_1.A4 (VBUS), USBC_IN_1.A9 (VBUS), USBC_IN_1.B4 (VBUS), USBC_IN_1.B9 (VBUS), USBC_OUT_1.A4 (VBUS), USBC_OUT_1.A9 (VBUS), USBC_OUT_1.B4 (VBUS), USBC_OUT_1.B9 (VBUS); no longer C2.2, C4.2, C8.1
- net at U2.4 (PORT): now also R8.2
- new net: R11.2, U1.4 (PORT)
- new net: R10.1, U1.3 (CURRENT_MODE)
- new net: C23.2, U1.21 (TX2p)
- new net: C8.2, U2.16 (TX1n)
- new net: C24.2, U1.20 (TX2n)
- new net: R9.2, U1.5 (VBUS_DET)
- new net: R12.2, U1.11 (DIR)
- new net: C9.1, U2.17 (TX1p)
- new net USBC_OUT_CC1: U1.2 (CC1), USBC_OUT_1.A5 (CC1)
- new net USBC_OUT_CC2: U1.1 (CC2), USBC_OUT_1.B5 (CC2)
- new net USBC_OUT_RXN1: U1.14 (RX1n), USBC_OUT_1.B10 (SSRXn1)
- new net USBC_OUT_RXN2: U1.18 (RX2n), USBC_OUT_1.A10 (SSRXn2)
- new net USBC_OUT_RXP1: U1.15 (RX1p), USBC_OUT_1.B11 (SSRXp1)
- new net USBC_OUT_RXP2: U1.19 (RX2p), USBC_OUT_1.A11 (SSRXp2)
- new net USBC_OUT_TXN1: U1.16 (TX1n), USBC_OUT_1.A3 (SSTXn1)
- new net USBC_OUT_TXN2: C24.1, USBC_OUT_1.B3 (SSTXn2)
- new net USBC_OUT_TXP1: U1.17 (TX1p), USBC_OUT_1.A2 (SSTXp1)
- new net USBC_OUT_TXP2: C23.1, USBC_OUT_1.B2 (SSTXp2)
- no-connect marks 51 -> 58
Other:
- moved on the sheet: C10, C11, C12, C13, C14, C15, C16, C17, C18, C20, C21, C22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

Commit message: BIG UPDATEEEEEEEEE
Parts:
- added C25: CC0603JRNPO9BN390, EasyEDA:C0603, symbol EasyEDA:CC0603JRNPO9BN390
- added R2: RC0402FR-0710KL, EasyEDA:R0402, symbol EasyEDA:RC0402FR-0710KL
Connections:
- net GND: now also USBC_IN_1.0 (EH), C25.2
- net VBUS: now also R2.2
- net at USB_CONTROLLER1.24 (RESETJ): now also R2.1
- net at USB_CONTROLLER1.45 (X1), X2.1 (OSC1): now also C25.1
- no-connect marks 58 -> 60
